Commit message: fix inconsistency in env
Signed-off-by: youliang <tan_you_liang@hotmail.com>

File: tennisbot/resources/court.urdf (robot description, URDF)
Before this commit: robot court, 1 links, 0 joints
Links:
- link base_link: geometry collision box size=20 20 0.01; collision box size=28 14 0.01

Commit message: small modifs;

File: tennisbot/resources/court.urdf (robot description, URDF)
Before this commit: robot court, 1 links, 0 joints
Links:
- link base_link: geometry collision box size=0.194382 12.6506 1; collision box size=28 14 0.01
